File: switch_matrix.kicad_sch (KiCad schematic)
At the start: 8 parts, among them SW1 MX_SW_solder, SW2 MX_SW_solder, SW3 MX_SW_solder, SW4 MX_SW_solder

Commit message: Updated LCSC part numbers for all parts.
Parts:
- D1, D2, D3, D4: footprint (none) -> Diode_SMD:D_SOD-123; LCSC (none) -> C81598
Changed lines of the file:
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@@
       (effects (font (size 1.27 1.27)) (justify right))
     )
-    (property "Footprint" "" (at 85.09 43.18 90)
+    (property "Footprint" "Diode_SMD:D_SOD-123" (at 85.09 43.18 90)
       (effects (font (size 1.27 1.27)) hide)
     )
@@
       (effects (font (size 1.27 1.27)) hide)
     )
+    (property "LCSC" "C81598" (at 85.09 43.18 0)
+      (effects (font (size 1.27 1.27)) hide)
+    )
     (pin "1")
     (pin "2")
@@
       (effects (font (size 1.27 1.27)) (justify right))
     )
-    (property "Footprint" "" (at 59.69 62.23 90)
+    (property "Footprint" "Diode_SMD:D_SOD-123" (at 59.69 62.23 90)
       (effects (font (size 1.27 1.27)) hide)
     )
@@
       (effects (font (size 1.27 1.27)) hide)
     )
+    (property "LCSC" "C81598" (at 59.69 62.23 0)
+      (effects (font (size 1.27 1.27)) hide)
+    )
     (pin "1")
     (pin "2")
@@
       (effects (font (size 1.27 1.27)) (justify right))
     )
-    (property "Footprint" "" (at 59.69 43.18 90)
+    (property "Footprint" "Diode_SMD:D_SOD-123" (at 59.69 43.18 90)
       (effects (font (size 1.27 1.27)) hide)
     )
@@
       (effects (font (size 1.27 1.27)) hide)
     )
+    (property "LCSC" "C81598" (at 59.69 43.18 0)
+      (effects (font (size 1.27 1.27)) hide)
+    )
     (pin "1")
     (pin "2")
@@
       (effects (font (size 1.27 1.27)) (justify right))
     )
-    (property "Footprint" "" (at 85.09 62.23 90)
+    (property "Footprint" "Diode_SMD:D_SOD-123" (at 85.09 62.23 90)
       (effects (font (size 1.27 1.27)) hide)
     )
@@
       (effects (font (size 1.27 1.27)) hide)
     )
+    (property "LCSC" "C81598" (at 85.09 62.23 0)
+      (effects (font (size 1.27 1.27)) hide)
+    )
